File: YauDL.sch (KiCad schematic (older format))
At the start: 0 parts

Commit message: Schematic work.
Parts:
- added C1, C2: CP1, symbol CP1
- added D1: DIODESCH, symbol DIODESCH
- added K1: HEATSINK, symbol CONN_3
- added MH1, MH2, MH3, MH4, P1, P2: CONN_1, symbol CONN_1
- added Q1, Q2: IRLZ34N, symbol MADW__IRLZ34N
- added R1, R2, R3, R4: R, symbol R
- added RV1, RV2: 100k, symbol POT
- added U1: TS2940, symbol TS2940
- added U2: MADW__LM2904, symbol MADW__LM2904
Connections:
- net labels added: GND, GNDPWR, VCC, V_in, drain
- wire segments 0 -> 66
- no-connect marks 0 -> 7
Other:
- note added: "1V / 1A"
- note added: "DUT input"
- note added: "FOLLOW"
- note added: "GAIN"
- note added: "min. 5A cont."

Commit message: Doodles...
Parts:
- removed D1: DIODESCH, symbol DIODESCH
- removed U1: TS2940, symbol TS2940
- added BT1: BATTERY, symbol BATTERY
- added DZ1: VZ10, symbol MADW__ZENER_SOT23
- added Q3, Q4: AO3401, symbol MOSFET_P
- added R1: 0R, symbol R
- added R2, R9: 100k, symbol R
- added R7, R8: 10k 0.1%, symbol R
- added T3, T4: Banana socket, symbol CONN_1
- added U1: AMS1117, symbol MADW__AMS1117
- added unit 3 of U2
- C1, C2: value CP1 -> 10µF
- R3: renamed from R1; value R -> 0.22R 5%
- R4: renamed from R2; value R -> 0.22R 5%
- R5: renamed from R3; value R -> 0.22R 5%
- R6: renamed from R4; value R -> 0.22R 5%
- T1: renamed from P1; value CONN_1 -> Binding post
- T2: renamed from P2; value CONN_1 -> Binding post
- U2: value MADW__LM2904 -> LM2904
Connections:
- net labels added: DMM_read, V_ref, rp_prot, source
- net labels removed: V_in
- wire segments 66 -> 96
Other:
- note added: "(0.5V/1A)"
- note added: "(0.6W)"
- note added: "(1V/1A)"
- note added: "(3.3V)"
- note added: "(FOLLOW)"
- note added: "(GAIN)"
- note added: "DMM output"
- note added: "DUT reverse polarity protection"
- note removed: "1V / 1A"
- note removed: "FOLLOW"
- note removed: "GAIN"
- note removed: "min. 5A cont."
- moved on the sheet: K1, Q1, Q2, R3, R4, R5, R6, RV1, RV2, T1, T2, U2A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

Commit message: Doodles.
Parts:
- removed R7: 10k 0.1%, symbol R
- removed U1: AMS1117, symbol MADW__AMS1117
- added C3: 100nF, symbol C
- added D1: LED, symbol LED
- added SW1: SWITCH_INV, symbol SWITCH_INV
- added U1: TS2940, symbol TS2940
- BT1: value BATTERY -> 9V
- DZ1: value VZ10 -> BZX84C-10
- R8: value 10k 0.1% -> 1k
- renumbered R9 to R7
Connections:
- net DMM_read: now also U2.6 (2IN-), C3.1
- net GND: now also MH1.1, MH2.1, MH3.1, MH4.1, D1.2 (K), SW1.1, U1.2 (GND); no longer BT1.2 (-), R7.2, R8.2
- net GNDPWR: now also R7.2
- net VCC: now also U1.1 (IN)
- net V_ref: now also R8.2, U1.3 (OUT)
- net at RV1.2, U2.2 (1IN-): now also C3.2
- net at R8.1: now also D1.1 (A); no longer U2.6 (2IN-)
- new net: BT1.2 (-), SW1.2
- no-connect marks 7 -> 4
Other:
- note added: "(10-turn Pot.)\n"
- note added: "(5V)"
- note added: "(BW limit)"
- note added: "(Trimmer: GAIN)"
- note removed: "(0.5V/1A)"
- note removed: "(3.3V)"
- note removed: "(GAIN)"
- moved on the sheet: BT1, C1, C2, DZ1, K1, MH1, MH2, MH3, MH4, Q1, Q2, Q3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

Commit message: Done?
Parts:
- BT1: value 9V -> 9V battery
Changed lines of the file:
@@
-EESchema Schematic File Version 2  date Mon 04 Jun 2012 05:08:03 PM CEST
+EESchema Schematic File Version 2  date Tue 05 Jun 2012 09:27:59 AM CEST
 LIBS:my_parts
 LIBS:power
@@
 Sheet 1 1
 Title "(Yet) (a)nother (u)seless (D)ummy (Load) - YauDL"
-Date "4 jun 2012"
+Date "5 jun 2012"
 Rev "0.1"
 Comp "2012 - My 2muF - blog.spitzenpfeil.org"
@@
 P 1250 3500
 F 0 "BT1" H 1250 3700 50  0000 C CNN
-F 1 "9V" H 1250 3310 50  0000 C CNN
+F 1 "9V battery" H 1250 3310 50  0000 C CNN
 	1    1250 3500
 	-1   0    0    1
