File: YauDL.kicad_pcb (KiCad board)
At the start: 2 copper layers, 100 x 100 mm, 49 parts, among them P1 REMOTE, Q1 IRL3803, Q2 IRL3803, SW1 SWITCH_INV, T1 Binding_post, T2 Binding_post, T3 Binding_post, T4 Binding_post, U1 TS2940, U2 LM2904

Commit message: Fixed missing module definitions (pcbnew BZR 4319 was barfing).
Parts:
- G1, G2: value LOGO -> LED_SMILE; footprint LOGO -> LED_SMILE
- G3, G4: value LOGO -> OSHW_LOGO; footprint (none) -> OSHW_LOGO
- G5, G6: value LOGO -> FIRE; footprint LOGO -> FIRE
- G7, G8: value LOGO -> CHINESE_ORDER_NUMBER; footprint LOGO -> CHINESE_ORDER_NUMBER
Changed lines of the file:
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@@
-(kicad_pcb (version 3) (host pcbnew "(2013-06-27 BZR 4227)-testing")
+(kicad_pcb (version 3) (host pcbnew "(2013-09-16 BZR 4319)-product")
   (general
     (links 68)
@@
     (pad_to_mask_clearance 0)
     (aux_axis_origin 0 0)
-    (visible_elements FFFFFFBF)
+    (visible_elements FFFFFFFF)
     (pcbplotparams
       (layerselection 351305729)
@@
     )
   )
-  (module LOGO (layer Front)
+  (module CHINESE_ORDER_NUMBER (layer Front)
     (at 124.968 59.69)
-    (path LOGO)
     (fp_text reference G7 (at 0 2.51968) (layer F.SilkS) hide
       (effects (font (size 0.43942 0.43942) (thickness 0.08636)))
     )
-    (fp_text value LOGO (at 0 -2.51968) (layer F.SilkS) hide
+    (fp_text value CHINESE_ORDER_NUMBER (at 0 -2.51968) (layer F.SilkS) hide
       (effects (font (size 0.43942 0.43942) (thickness 0.08636)))
     )
@@
       (xy -10.56894 -0.78232)) (layer F.SilkS) (width 0.00254))
   )
-  (module LOGO (layer Front)
+  (module CHINESE_ORDER_NUMBER (layer Front)
     (at 165.1 59.69)
-    (path LOGO)
     (fp_text reference G8 (at 0 2.51968) (layer F.SilkS) hide
       (effects (font (size 0.43942 0.43942) (thickness 0.08636)))
     )
-    (fp_text value LOGO (at 0 -2.51968) (layer F.SilkS) hide
+    (fp_text value CHINESE_ORDER_NUMBER (at 0 -2.51968) (layer F.SilkS) hide
       (effects (font (size 0.43942 0.43942) (thickness 0.08636)))
     )
@@
       (xy -10.56894 -0.78232)) (layer F.SilkS) (width 0.00254))
   )
-  (module "" (layer Front)
+  (module OSHW_LOGO (layer Front)
     (at 175.00092 38.99916)
     (fp_text reference G3 (at 0 4.72186) (layer F.SilkS) hide
       (effects (font (size 0.4064 0.4064) (thickness 0.08128)))
     )
-    (fp_text value LOGO (at 0 -4.72186) (layer F.SilkS) hide
+    (fp_text value OSHW_LOGO (at 0 -4.72186) (layer F.SilkS) hide
       (effects (font (size 0.4064 0.4064) (thickness 0.08128)))
     )
@@
       (xy -2.69748 3.99796)) (layer F.SilkS) (width 0.00254))
   )
-  (module "" (layer Back)
+  (module OSHW_LOGO (layer Back)
     (at 175.00092 38.99916)
     (fp_text reference G4 (at 0 -4.72186) (layer B.SilkS) hide
       (effects (font (size 0.4064 0.4064) (thickness 0.08128)) (justify mirror))
     )
-    (fp_text value LOGO (at 0 4.72186) (layer B.SilkS) hide
+    (fp_text value OSHW_LOGO (at 0 4.72186) (layer B.SilkS) hide
       (effects (font (size 0.4064 0.4064) (thickness 0.08128)) (justify mirror))
     )
@@
     )
   )
-  (module LOGO (layer Front)
+  (module FIRE (layer Front)
     (at 186.055 49.911)
-    (path LOGO)
     (fp_text reference G6 (at 0 4.2164) (layer F.SilkS) hide
       (effects (font (size 0.14224 0.14224) (thickness 0.02794)))
     )
-    (fp_text value LOGO (at 0 -4.2164) (layer F.SilkS) hide
+    (fp_text value FIRE (at 0 -4.2164) (layer F.SilkS) hide
       (effects (font (size 0.14224 0.14224) (thickness 0.02794)))
     )
@@
       (xy 2.99974 0.6096) (xy 3.00228 0.6096) (xy 3.00228 0.6096)) (layer F.SilkS) (width 0.00254))
   )
-  (module LOGO (layer Front)
+  (module FIRE (layer Front)
     (at 104.14 50.038)
-    (path LOGO)
     (fp_text reference G5 (at 0 4.2164) (layer F.SilkS) hide
       (effects (font (size 0.14224 0.14224) (thickness 0.02794)))
     )
-    (fp_text value LOGO (at 0 -4.2164) (layer F.SilkS) hide
+    (fp_text value FIRE (at 0 -4.2164) (layer F.SilkS) hide
       (effects (font (size 0.14224 0.14224) (thickness 0.02794)))
     )
@@
       (xy 2.99974 0.6096) (xy 3.00228 0.6096) (xy 3.00228 0.6096)) (layer F.SilkS) (width 0.00254))
   )
-  (module LOGO (layer Back)
+  (module LED_SMILE (layer Back)
     (at 115.00104 38.99916)
-    (path LOGO)
     (fp_text reference G2 (at 0 -4.58978) (layer B.SilkS) hide
       (effects (font (size 0.127 0.127) (thickness 0.02032)) (justify mirror))
     )
-    (fp_text value LOGO (at 0 4.58978) (layer B.SilkS) hide
+    (fp_text value LED_SMILE (at 0 4.58978) (layer B.SilkS) hide
       (effects (font (size 0.127 0.127) (thickness 0.02032)) (justify mirror))
     )
@@
       (xy 1.3081 -1.52654) (xy 1.40716 -1.4986) (xy 1.41732 -1.4986) (xy 1.51892 -1.49098)) (layer B.SilkS) (width 0.00254))
   )
-  (module LOGO (layer Front)
+  (module LED_SMILE (layer Front)
     (at 115.00104 38.99916)
-    (path LOGO)
     (fp_text reference G1 (at 0 4.58978) (layer F.SilkS) hide
       (effects (font (size 0.127 0.127) (thickness 0.02032)))
     )
-    (fp_text value LOGO (at 0 -4.58978) (layer F.SilkS) hide
+    (fp_text value LED_SMILE (at 0 -4.58978) (layer F.SilkS) hide
       (effects (font (size 0.127 0.127) (thickness 0.02032)))
     )
